Commit message: docs: 補齊 01/02/03/04/07/28 章的圖，並修正 04 章模型的三個錯誤
到這裡每個實驗章節都有圖了。

04 章的模型本身是錯的（渲染出來才發現）：
- <visual> 被整組丟掉：discardvisual 對 URDF 的預設是 true，不是文件寫的 false。
  不明寫 false 就只剩 collision 幾何，模型照樣載入、照樣模擬，只是長得不對
- 圓柱軸向錯 90°：rpy="1.5707963 0 0" 讓沿 z 的圓柱橫躺，但關節是沿 z 排列的，
  於是畫面上是兩根分離的短棒
- 修正軸向後手臂被彈飛：連桿頂端伸進固定底座 50 mm，1 秒內 1899 次假接觸。
  底座併進 world 之後父子碰撞排除不涵蓋它，而關節就在底座表面上 —— 縮短連桿的
  collision 沒有用，底座不給 <collision> 才是解

修好之後 1 秒後的 qpos 回到 [-0.637, -0.802]，與修正前完全相同：原本橫躺的錯誤
幾何意外避開了那個碰撞，所以動力學一直是對的，只有畫面不對。沒有人渲染過它。

順帶查證：URDF 的 <mujoco> 區段只吃 compiler / option / size，寫 <default> 或
<contact> 會被靜默忽略（實測 nexclude = 0），官方文件明說連 MuJoCo 專屬元素也不做
schema 檢查。

新增的圖：
- 03 章 PD 控制：響應曲線 ＋ KP 掃描（穩態誤差 14.6° → 0.3°，永遠不歸零）
- 07 章三個範例：接觸力尖峰（200 Hz 才抓得到）、伺服的相位落後、16 條 rollout 發散
- 01/02/04 章模型外觀，04 章另有 visual / collision 的分組對照
- 28 章吞吐長條圖

新增 make_model_figures.py（從模型檔直接渲染）。踩到的坑：剛建立的 mjData 直接
渲染會得到全黑的一格，要先 mj_forward —— 而且只有 t=0 那格黑，後面的因為 mj_step
算過就正常，很容易誤判成「第一次渲染的已知問題」。

Co-Authored-By: Claude Opus 5 (1M context) <noreply@anthropic.com>

File: models/two_link_arm.urdf (robot description, URDF)
Before this commit: robot two_link_arm, 3 links, 2 joints
Links:
- link base: geometry visual box size=0.1 0.1 0.05
